Commit message: add gazebo files

File: xy_unilivers_description/urdf/xy_unilivers.urdf_with_gazebo_color.xacro (robot description, xacro)
@@ -2,12 +2,7 @@
 <robot xmlns:xacro="http://www.ros.org/wiki/xacro" name="xy_unilivers">
   <link name="world" />
-  <!-- Used for fixing robot -->
-  <gazebo reference="world">
-    <static>true</static>
-  </gazebo>
   <joint name="world_to_base" type="fixed">
     <parent link="world" />
     <child link="base" />
-    <origin xyz="0. 0. 0.25" rpy="0 0 0" />
   </joint>
   <link name="base">
@@ -17,5 +12,5 @@
           scale="0.001 0.001 0.001" />
       </geometry>
-      <origin xyz="0 0 0.0" rpy="0 0 ${radians(90)}" />
+      <origin xyz="0 0 0" rpy="0 0 ${radians(90)}" />
       <material name="grey">
         <color rgba="0.4 0.4 0.4 1." />
@@ -24,5 +19,5 @@
     <!--TODO provides accurate values for the inertial tags = following values are arbitrary-->
     <inertial>
-      <mass value="10" />
+      <mass value="1" />
       <inertia ixx="1e-3" ixy="0.0" ixz="0.0" iyy="1e-3" iyz="0.0" izz="1e-3" />
     </inertial>
@@ -49,27 +44,18 @@
       </material>
     </visual>
-    <collision name="charriot_collision">
+    <collision>
       <geometry>
         <mesh filename="package://xy_unilivers_description/meshes/charriot.stl"
           scale="0.001 0.001 0.001" />
       </geometry>
-      <origin xyz="0.075 0.0 0.0" rpy="${radians(-90)} 0 0" />
     </collision>
     <!--TODO provides accurate values for the inertial tags = following values are arbitrary-->
     <inertial>
       <mass value="1" />
-      <origin xyz="22.234152e-3 -25.151773e-3 -1.542117e-3" />
-      <inertia ixx="6737.72608" ixy="99.53903" ixz="-137.44316" iyy="13064.48256" iyz="79.50954" izz="6989.75104" />
+      <inertia ixx="1e-3" ixy="0.0" ixz="0.0" iyy="1e-3" iyz="0.0" izz="1e-3" />
     </inertial>
   </link>
   <gazebo reference="charriot">
-    <gravity>true</gravity>
     <material>Gazebo/White</material>
-    <kp>1000000.0</kp>
-    <kd>1.0</kd>
-    <mu1>0.8</mu1>
-    <mu2>0.8</mu2>
-    <maxVel>0.5</maxVel>
-    <minDepth>0.0005</minDepth>
   </gazebo>
   <joint name="base_to_switch1" type="fixed">
@@ -89,10 +75,9 @@
       </material>
     </visual>
-    <collision name="switch1_left_collision">
+    <collision>
       <geometry>
         <mesh filename="package://xy_unilivers_description/meshes/switch.stl"
           scale="0.001 0.001 0.001" />
       </geometry>
-      <origin xyz="0.0 0.0 0.0" rpy="0 0 0" />
     </collision>
     <!--TODO provides accurate values for the inertial tags = following values are arbitrary-->
@@ -104,10 +89,4 @@
   <gazebo reference="switch1">
     <material>Gazebo/Green</material>
-    <kp>1000000.0</kp>
-    <kd>1.0</kd>
-    <mu1>0.8</mu1>
-    <mu2>0.8</mu2>
-    <maxVel>0.5</maxVel>
-    <minDepth>0.0005</minDepth>
   </gazebo>
   <joint name="base_to_switch2" type="fixed">
@@ -128,10 +107,9 @@
       </material>
     </visual>
-    <collision name="switch2_right_collision">
+    <collision>
       <geometry>
         <mesh filename="package://xy_unilivers_description/meshes/switch.stl"
           scale="0.001 0.001 0.001" />
       </geometry>
-      <origin xyz="0.0 0.0 0.0" rpy="0 0 0" />
     </collision>
     <!--TODO provides accurate values for the inertial tags = following values are arbitrary-->
@@ -143,78 +121,8 @@
   <gazebo reference="switch2">
     <material>Gazebo/Blue</material>
-    <kp>1000000.0</kp>
-    <kd>1.0</kd>
-    <mu1>0.8</mu1>
-    <mu2>0.8</mu2>
-    <maxVel>0.5</maxVel>
-    <minDepth>0.0005</minDepth>
   </gazebo>
-  <gazebo>
-    <plugin name="gazebo_ros_joint_state_publisher"
-            filename="libgazebo_ros_joint_state_publisher.so">
-      <update_rate>20</update_rate>
-      <joint_name>base_to_charriot</joint_name>
-    </plugin>
-  </gazebo>
-  <gazebo>
-    <plugin name="gazebo_ros_joint_pose_trajectory"
-        filename="libgazebo_ros_joint_pose_trajectory.so">
-        <update_rate>20</update_rate>
-    </plugin>
-  </gazebo>
-  <!--contact sensor charriot-->
-  <gazebo reference="charriot">
-    <sensor name="switch1_contactsensor_sensor" type="contact">
-      <selfCollide>true</selfCollide>
-      <always_on>true</always_on>
-      <updateRate>1</updateRate>
-      <contact>
-        <collision>charriot_collision_collision</collision>
-      </contact>
-      <plugin name="charriot_bumper_plugin" filename="libgazebo_ros_bumper.so">
-        <ros>
-          <namespace>contact_sensor</namespace>
-          <remapping>bumper_states:=bumper_charriot</remapping>
-        </ros>
-        <frameName>charriot</frameName>
-      </plugin>
-    </sensor>
-  </gazebo>
-  <!--contact sensor switch1-->
-  <gazebo reference="switch1">
-    <sensor name="switch1_contactsensor_sensor" type="contact">
-      <selfCollide>true</selfCollide>
-      <always_on>true</always_on>
-      <updateRate>1</updateRate>
-      <contact>
-        <collision>base_fixed_joint_lump__switch1_left_collision_collision</collision>
-      </contact>
-      <plugin name="switch1_bumper_plugin" filename="libgazebo_ros_bumper.so">
-        <ros>
-          <namespace>contact_sensor</namespace>
-          <remapping>bumper_states:=bumper_switch1_left</remapping>
-        </ros>
-        <frameName>switch1</frameName>
-      </plugin>
-    </sensor>
-  </gazebo>
-  <!--contact sensor switch2-->
-  <gazebo reference="switch2">
-    <sensor name="switch2_contactsensor_sensor" type="contact">
-      <selfCollide>true</selfCollide>
-      <always_on>true</always_on>
-      <updateRate>1</updateRate>
-      <contact>
-        <collision>base_fixed_joint_lump__switch2_right_collision_collision_1</collision>
-      </contact>
-      <plugin name="switch2_bumper_plugin" filename="libgazebo_ros_bumper.so">
-        <ros>
-          <namespace>contact_sensor</namespace>
-          <remapping>bumper_states:=bumper_switch2_right</remapping>
-        </ros>
-        <bumperTopicName>switch2_right_contact</bumperTopicName>
-        <frameName>switch2</frameName>
-      </plugin>
-    </sensor>
-  </gazebo>
+  <!-- Used for fixing robot -->
+    <gazebo reference="world">
+        <static>true</static>
+    </gazebo>
 </robot>
