Commit message: Simple velocity controller ok.

File: xy_unilivers_description/urdf/xy_unilivers.urdf.xacro (robot description, xacro)
@@ -1,4 +1,9 @@
 <?xml version="1.0"?>
 <robot xmlns:xacro="http://www.ros.org/wiki/xacro" name="xy_unilivers">
+  <link name="world" />
+  <joint name="world_to_base_link" type="fixed">
+    <parent link="world" />
+    <child link="base_link" />
+  </joint>
   <link name="base_link">
     <visual>
@@ -15,10 +20,10 @@
   <joint name="base_to_charriot" type="prismatic">
     <parent link="base_link" />
-    <child link="Charriot" />
-    <origin xyz="0.036 0 0" rpy="0 0 0" />
+    <child link="charriot" />
+    <origin xyz="-0.104 0 0" rpy="0 0 0" />
     <axis xyz="1 0 0" />
-    <limit lower="-0.178" upper="-0.03" effort="1000" velocity="0.5" />
+    <limit lower="-0.037" upper="0.110" effort="1000" velocity="0.5" />
   </joint>
-  <link name="Charriot">
+  <link name="charriot">
     <visual>
       <geometry>
@@ -31,4 +36,15 @@
       </material>
     </visual>
+    <collision>
+      <geometry>
+        <mesh filename="package://xy_unilivers_description/meshes/charriot.stl"
+          scale="0.001 0.001 0.001" />
+      </geometry>
+    </collision>
+    <!--TODO provides accurate values for the inertial tags = following values are arbitrary-->
+    <inertial>
+      <mass value="1" />
+      <inertia ixx="1e-3" ixy="0.0" ixz="0.0" iyy="1e-3" iyz="0.0" izz="1e-3" />
+    </inertial>
   </link>
   <joint name="base_to_switch1" type="fixed">
@@ -48,4 +64,10 @@
       </material>
     </visual>
+    <collision>
+      <geometry>
+        <mesh filename="package://xy_unilivers_description/meshes/switch.stl"
+          scale="0.001 0.001 0.001" />
+      </geometry>
+    </collision>
   </link>
   <joint name="base_to_switch2" type="fixed">
@@ -66,4 +88,10 @@
       </material>
     </visual>
+    <collision>
+      <geometry>
+        <mesh filename="package://xy_unilivers_description/meshes/switch.stl"
+          scale="0.001 0.001 0.001" />
+      </geometry>
+    </collision>
   </link>
 </robot>

Commit message: Add gazebo simulation.

File: xy_unilivers_description/urdf/xy_unilivers.urdf.xacro (robot description, xacro)
@@ -2,9 +2,14 @@
 <robot xmlns:xacro="http://www.ros.org/wiki/xacro" name="xy_unilivers">
   <link name="world" />
-  <joint name="world_to_base_link" type="fixed">
+  <!-- Used for fixing robot -->
+  <gazebo reference="world">
+    <static>true</static>
+  </gazebo>
+  <joint name="world_to_base" type="fixed">
     <parent link="world" />
-    <child link="base_link" />
-  </joint>
-  <link name="base_link">
+    <child link="base" />
+    <origin xyz="0. 0. 0.25" rpy="0 0 0" />
+  </joint>
+  <link name="base">
     <visual>
       <geometry>
@@ -12,12 +17,20 @@
           scale="0.001 0.001 0.001" />
       </geometry>
-      <origin xyz="0 0 0" rpy="0 0 ${radians(90)}" />
+      <origin xyz="0 0 0.0" rpy="0 0 ${radians(90)}" />
       <material name="grey">
         <color rgba="0.4 0.4 0.4 1." />
       </material>
     </visual>
-  </link>
+    <!--TODO provides accurate values for the inertial tags = following values are arbitrary-->
+    <inertial>
+      <mass value="10" />
+      <inertia ixx="1e-3" ixy="0.0" ixz="0.0" iyy="1e-3" iyz="0.0" izz="1e-3" />
+    </inertial>
+  </link>
+  <gazebo reference="base">
+    <material>Gazebo/Grey</material>
+  </gazebo>
   <joint name="base_to_charriot" type="prismatic">
-    <parent link="base_link" />
+    <parent link="base" />
     <child link="charriot" />
     <origin xyz="-0.104 0 0" rpy="0 0 0" />
@@ -36,18 +49,39 @@
       </material>
     </visual>
-    <collision>
+    <collision name="charriot_collision">
       <geometry>
         <mesh filename="package://xy_unilivers_description/meshes/charriot.stl"
           scale="0.001 0.001 0.001" />
       </geometry>
+      <origin xyz="0.075 0.0 0.0" rpy="${radians(-90)} 0 0" />
+      <surface>
+        <friction> <ode> <mu>mu1</mu> <mu2>m2</mu2> </ode> </friction>
+        <contact>
+          <!--
+          <collide_bitmask>0x10000</collide_bitmask>
+          -->
+          <ode> <kp>kp</kp> <kd>kd</kd> </ode>
+        </contact>
+      </surface>
     </collision>
     <!--TODO provides accurate values for the inertial tags = following values are arbitrary-->
     <inertial>
       <mass value="1" />
-      <inertia ixx="1e-3" ixy="0.0" ixz="0.0" iyy="1e-3" iyz="0.0" izz="1e-3" />
-    </inertial>
-  </link>
+      <origin xyz="22.234152e-3 -25.151773e-3 -1.542117e-3" />
+      <inertia ixx="6737.72608" ixy="99.53903" ixz="-137.44316" iyy="13064.48256" iyz="79.50954" izz="6989.75104" />
+    </inertial>
+  </link>
+  <gazebo reference="charriot">
+    <gravity>true</gravity>
+    <material>Gazebo/White</material>
+    <kp>1000000.0</kp>
+    <kd>1.0</kd>
+    <mu1>0.8</mu1>
+    <mu2>0.8</mu2>
+    <maxVel>0.5</maxVel>
+    <minDepth>0.0005</minDepth>
+  </gazebo>
   <joint name="base_to_switch1" type="fixed">
-    <parent link="base_link" />
+    <parent link="base" />
     <child link="switch1" />
     <origin xyz="${0.003-0.08} ${-0.051} -0.002" rpy="${radians(90)} ${radians(-90)} 0" />
@@ -64,13 +98,37 @@
       </material>
     </visual>
-    <collision>
-      <geometry>
-        <mesh filename="package://xy_unilivers_description/meshes/switch.stl"
-          scale="0.001 0.001 0.001" />
-      </geometry>
+    <collision name="switch1_left_collision">
+      <geometry>
+        <mesh filename="package://xy_unilivers_description/meshes/switch.stl"
+          scale="0.001 0.001 0.001" />
+      </geometry>
+      <origin xyz="0.0 0.0 0.0" rpy="0 0 0" />
+      <surface>
+        <friction> <ode> <mu>mu1</mu> <mu2>m2</mu2> </ode> </friction>
+        <contact>
+          <!--
+          <collide_bitmask>0x10000</collide_bitmask>
+          -->
+          <ode> <kp>kp</kp> <kd>kd</kd> </ode>
+        </contact>
+      </surface>
     </collision>
-  </link>
+    <!--TODO provides accurate values for the inertial tags = following values are arbitrary-->
+    <inertial>
+      <mass value="0.1" />
+      <inertia ixx="1e-3" ixy="0.0" ixz="0.0" iyy="1e-3" iyz="0.0" izz="1e-3" />
+    </inertial>
+  </link>
+  <gazebo reference="switch1">
+    <material>Gazebo/Green</material>
+    <kp>1000000.0</kp>
+    <kd>1.0</kd>
+    <mu1>0.8</mu1>
+    <mu2>0.8</mu2>
+    <maxVel>0.5</maxVel>
+    <minDepth>0.0005</minDepth>
+  </gazebo>
   <joint name="base_to_switch2" type="fixed">
-    <parent link="base_link" />
+    <parent link="base" />
     <child link="switch2" />
     <origin xyz="${0.089+0.005} ${-0.051} ${-0.002}"
@@ -88,10 +146,102 @@
       </material>
     </visual>
-    <collision>
-      <geometry>
-        <mesh filename="package://xy_unilivers_description/meshes/switch.stl"
-          scale="0.001 0.001 0.001" />
-      </geometry>
+    <collision name="switch2_right_collision">
+      <geometry>
+        <mesh filename="package://xy_unilivers_description/meshes/switch.stl"
+          scale="0.001 0.001 0.001" />
+      </geometry>
+      <origin xyz="0.0 0.0 0.0" rpy="0 0 0" />
+      <surface>
+        <friction> <ode> <mu>mu1</mu> <mu2>m2</mu2> </ode> </friction>
+        <contact>
+          <!--
+          <collide_bitmask>0x10000</collide_bitmask>
+          -->
+          <ode> <kp>kp</kp> <kd>kd</kd> </ode>
+        </contact>
+      </surface>
     </collision>
-  </link>
+    <!--TODO provides accurate values for the inertial tags = following values are arbitrary-->
+    <inertial>
+      <mass value="0.1" />
+      <inertia ixx="1e-3" ixy="0.0" ixz="0.0" iyy="1e-3" iyz="0.0" izz="1e-3" />
+    </inertial>
+  </link>
+  <gazebo reference="switch2">
+    <material>Gazebo/Blue</material>
+    <kp>1000000.0</kp>
+    <kd>1.0</kd>
+    <mu1>0.8</mu1>
+    <mu2>0.8</mu2>
+    <maxVel>0.5</maxVel>
+    <minDepth>0.0005</minDepth>
+  </gazebo>
+  <gazebo>
+    <plugin name="gazebo_ros_joint_state_publisher"
+            filename="libgazebo_ros_joint_state_publisher.so">
+      <update_rate>20</update_rate>
+      <joint_name>base_to_charriot</joint_name>
+    </plugin>
+  </gazebo>
+  <gazebo>
+    <plugin name="gazebo_ros_joint_pose_trajectory"
+        filename="libgazebo_ros_joint_pose_trajectory.so">
+        <update_rate>20</update_rate>
+    </plugin>
+  </gazebo>
+  <!--contact sensor charriot-->
+  <gazebo reference="charriot">
+    <sensor name="switch1_contactsensor_sensor" type="contact">
+      <selfCollide>true</selfCollide>
+      <always_on>true</always_on>
+      <updateRate>1</updateRate>
+      <contact>
+        <collision>charriot_collision_collision</collision>
+      </contact>
+      <plugin name="charriot_bumper_plugin" filename="libgazebo_ros_bumper.so">
+        <ros>
+          <namespace>contact_sensor</namespace>
+          <remapping>bumper_states:=bumper_charriot</remapping>
+        </ros>
+        <frameName>charriot</frameName>
+      </plugin>
+    </sensor>
+  </gazebo>
+  <!--contact sensor switch1-->
+  <gazebo reference="switch1">
+    <sensor name="switch1_contactsensor_sensor" type="contact">
+      <selfCollide>true</selfCollide>
+      <always_on>true</always_on>
+      <updateRate>1</updateRate>
+      <contact>
+        <collision>base_fixed_joint_lump__switch1_left_collision_collision</collision>
+      </contact>
+      <plugin name="switch1_bumper_plugin" filename="libgazebo_ros_bumper.so">
+        <ros>
+          <namespace>contact_sensor</namespace>
+          <remapping>bumper_states:=bumper_switch1_left</remapping>
+        </ros>
+        <frameName>switch1</frameName>
+      </plugin>
+    </sensor>
+  </gazebo>
+  <!--contact sensor switch2-->
+  <gazebo reference="switch2">
+    <sensor name="switch2_contactsensor_sensor" type="contact">
+      <selfCollide>true</selfCollide>
+      <always_on>true</always_on>
+      <updateRate>1</updateRate>
+      <contact>
+        <collision>base_fixed_joint_lump__switch2_right_collision_collision_1</collision>
+      </contact>
+      <plugin name="switch2_bumper_plugin" filename="libgazebo_ros_bumper.so">
+        <ros>
+          <namespace>contact_sensor</namespace>
+          <remapping>bumper_states:=bumper_switch2_right</remapping>
+        </ros>
+        <bumperTopicName>switch2_right_contact</bumperTopicName>
+        <frameName>switch2</frameName>
+      </plugin>
+    </sensor>
+  </gazebo>
 </robot>

File: xy_unilivers_description/urdf/xy_unilivers_simplified.urdf (robot description, URDF)
Before this commit: robot xy_unilivers, 2 links, 1 joints
Links:
- removed link base_link
- added link base; visual box size=0.80 0.10 0.22
Joints:
- joint base_to_charriot: parent base_link -> base

Commit message: Fix collision detection between switch and charriot

File: xy_unilivers_description/urdf/xy_unilivers.urdf.xacro (robot description, xacro)
@@ -73,8 +73,10 @@
     <minDepth>0.0005</minDepth>
   </gazebo>
-  <joint name="base_to_switch1" type="fixed">
+  <joint name="base_to_switch1" type="revolute">
     <parent link="base" />
     <child link="switch1" />
     <origin xyz="${0.003-0.08} ${-0.051} -0.002" rpy="${radians(90)} ${radians(-90)} 0" />
+    <axis xyz="0 0 1" />
+    <limit effort="0.0" lower="0.0" upper="0.0" velocity="0.0"/>
   </joint>
   <link name="switch1">
@@ -111,9 +113,11 @@
     <minDepth>0.0005</minDepth>
   </gazebo>
-  <joint name="base_to_switch2" type="fixed">
+  <joint name="base_to_switch2" type="revolute">
     <parent link="base" />
     <child link="switch2" />
     <origin xyz="${0.089+0.005} ${-0.051} ${-0.002}"
       rpy="${radians(90)} ${radians(90)} ${radians(0)}" />
+    <axis xyz="0 0 1" />
+    <limit effort="0.0" lower="0.0" upper="0.0" velocity="0.0"/>
   </joint>
   <link name="switch2">
@@ -153,5 +157,5 @@
     <plugin name="gazebo_ros_joint_state_publisher"
             filename="libgazebo_ros_joint_state_publisher.so">
-      <update_rate>20</update_rate>
+      <update_rate>1</update_rate>
       <joint_name>base_to_charriot</joint_name>
     </plugin>
@@ -160,16 +164,16 @@
     <plugin name="gazebo_ros_joint_pose_trajectory"
         filename="libgazebo_ros_joint_pose_trajectory.so">
-        <update_rate>20</update_rate>
+        <update_rate>1</update_rate>
     </plugin>
   </gazebo>
   <!--contact sensor charriot-->
   <gazebo reference="charriot">
-    <sensor name="switch1_contactsensor_sensor" type="contact">
-      <selfCollide>true</selfCollide>
+    <self_collide>1</self_collide>
+    <sensor name="charriot_contactsensor_sensor" type="contact">
       <always_on>true</always_on>
-      <updateRate>1</updateRate>
       <contact>
         <collision>charriot_collision_collision</collision>
       </contact>
+      <update_rate>1</update_rate>
       <plugin name="charriot_bumper_plugin" filename="libgazebo_ros_bumper.so">
         <ros>
@@ -177,5 +181,5 @@
           <remapping>bumper_states:=bumper_charriot</remapping>
         </ros>
-        <frameName>charriot</frameName>
+        <frame_name>charriot</frame_name>
       </plugin>
     </sensor>
@@ -183,11 +187,11 @@
   <!--contact sensor switch1-->
   <gazebo reference="switch1">
+    <self_collide>1</self_collide>
     <sensor name="switch1_contactsensor_sensor" type="contact">
-      <selfCollide>true</selfCollide>
       <always_on>true</always_on>
-      <updateRate>1</updateRate>
       <contact>
-        <collision>base_fixed_joint_lump__switch1_left_collision_collision</collision>
+        <collision>switch1_left_collision_collision</collision>
       </contact>
+      <update_rate>1</update_rate>
       <plugin name="switch1_bumper_plugin" filename="libgazebo_ros_bumper.so">
         <ros>
@@ -195,5 +199,5 @@
           <remapping>bumper_states:=bumper_switch1_left</remapping>
         </ros>
-        <frameName>switch1</frameName>
+        <frame_name>switch1</frame_name>
       </plugin>
     </sensor>
@@ -201,11 +205,11 @@
   <!--contact sensor switch2-->
   <gazebo reference="switch2">
+    <self_collide>1</self_collide>
     <sensor name="switch2_contactsensor_sensor" type="contact">
-      <selfCollide>true</selfCollide>
       <always_on>true</always_on>
-      <updateRate>1</updateRate>
       <contact>
-        <collision>base_fixed_joint_lump__switch2_right_collision_collision_1</collision>
+        <collision>switch2_right_collision_collision</collision>
       </contact>
+      <update_rate>1</update_rate>
       <plugin name="switch2_bumper_plugin" filename="libgazebo_ros_bumper.so">
         <ros>
@@ -213,6 +217,8 @@
           <remapping>bumper_states:=bumper_switch2_right</remapping>
         </ros>
+        <!--
         <bumperTopicName>switch2_right_contact</bumperTopicName>
-        <frameName>switch2</frameName>
+        -->
+        <frame_name>switch2</frame_name>
       </plugin>
     </sensor>

Commit message: Gazebo sim is now controlled with a slider using velocity command.

File: xy_unilivers_description/urdf/xy_unilivers.urdf.xacro (robot description, xacro)
@@ -36,5 +36,5 @@
     <origin xyz="-0.104 0 0" rpy="0 0 0" />
     <axis xyz="1 0 0" />
-    <limit lower="-0.037" upper="0.110" effort="1000" velocity="0.5" />
+    <limit lower="-0.037" upper="0.110" effort="1000" velocity="1.0" />
   </joint>
   <link name="charriot">
@@ -70,5 +70,5 @@
     <mu1>0.8</mu1>
     <mu2>0.8</mu2>
-    <maxVel>0.5</maxVel>
+    <maxVel>1.0</maxVel>
     <minDepth>0.0005</minDepth>
   </gazebo>
@@ -161,8 +161,21 @@
     </plugin>
   </gazebo>
+  <!-- gazebo joint_pose_trajectory command plugin
   <gazebo>
     <plugin name="gazebo_ros_joint_pose_trajectory"
         filename="libgazebo_ros_joint_pose_trajectory.so">
         <update_rate>1</update_rate>
+    </plugin>
+  </gazebo>
+  -->
+  <!-- gazebo velocity command plugin -->
+  <gazebo>
+    <plugin name="gazebo_ros_planar_move"
+        filename="libgazebo_ros_planar_move.so">
+        <update_rate>20</update_rate>
+        <command_topic>/cmd_vel</command_topic>
+        <odometry_topic>odom</odometry_topic>
+        <odometry_frame>odom</odometry_frame>
+        <robot_base_frame>base_to_charriot</robot_base_frame>
     </plugin>
   </gazebo>
