Commit message: gazebo with ros2_control is working

File: xy_unilivers_description/gazebo/xy_unilivers_ros2_control.gazebo.xacro (robot description, xacro)
@@ -7,6 +7,4 @@
         </hardware>
         <joint name="base_to_charriot">
-            <param name="mimic">base_to_charriot</param>
-            <param name="multiplier">1</param>
             <state_interface name="position" />
             <state_interface name="velocity" />

File: xy_unilivers_description/urdf/xy_unilivers_gazebo_ros2_control.urdf.xacro (robot description, xacro)
@@ -32,5 +32,4 @@
   </gazebo>
   <joint name="base_to_charriot" type="prismatic">
-    <mimic joint="base_to_charriot"/>
     <parent link="base" />
     <child link="charriot" />
